File: design/examples/kicad-slider/slider.kicad_pcb (KiCad board)
At the start: 2 copper layers, 20 x 54 mm, 26 parts, among them J1 Conn_Jacdac_CardEdge, J2 Conn_HackConnect, J3 Conn_Jacdac_CardEdge, U1 XC6206P332MR, U2 STM32G031FxPx

Commit message: Rename JD-PEC-01 to JC-PEC-02
Parts:
- J1, J3: footprint Connector_Jacdac:JD-PEC-01_Prerouted -> Connector_Jacdac:JD-PEC-02_Prerouted
Changed lines of the file:
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@@
       (net 1 GND))
   )
-  (module Connector_Jacdac:JD-PEC-01_Prerouted (layer B.Cu)
+  (module Connector_Jacdac:JD-PEC-02_Prerouted (layer B.Cu)
     (at 100 71 180)
     (descr "Jacdac edge connector with pre-routed connections between top and bottom layers. 0.29mm power and 0.22mm (~8 mil) data trace width, and 0.155mm (~6 mil) power and 0.25mm data trace clearance.")
@@
       (net 3 JD_PWR))
   )
-  (module Connector_Jacdac:JD-PEC-01_Prerouted (layer B.Cu)
+  (module Connector_Jacdac:JD-PEC-02_Prerouted (layer B.Cu)
     (at 100 125)
     (descr "Jacdac edge connector with pre-routed connections between top and bottom layers. 0.29mm power and 0.22mm (~8 mil) data trace width, and 0.155mm (~6 mil) power and 0.25mm data trace clearance.")
